Commit message: Need to close grip

File: poppy_ergo_jr.pybullet.urdf (robot description, URDF)
Before this commit: robot poppy_ergo_jr, 9 links, 8 joints
Links:
- link base_link: geometry collision cylinder length=0.03 radius=0.08
- link fixed_tip: geometry collision box size=0.020 0.025 0.003
- link long_U: geometry collision cylinder length=0.02 radius=0.02
- link moving_tip: geometry collision box size=0.003 0.025 0.02
- link section_1: geometry collision cylinder length=0.05 radius=0.02
- link section_2: geometry collision cylinder length=0.05 radius=0.02
- link section_3: geometry collision cylinder length=0.05 radius=0.02
- link section_4: geometry collision cylinder length=0.03 radius=0.02
- link section_5: geometry 

Commit message: Removed visual elements

File: poppy_ergo_jr.pybullet.urdf (robot description, URDF)
Before this commit: robot poppy_ergo_jr, 9 links, 8 joints
Links:
- link base_link: geometry collision cylinder length=0.03 radius=0.08; visual mesh filename=meshes/base.stl
- link fixed_tip: geometry collision box size=0.020 0.025 0.003; visual box size=0 0 0
- link long_U: geometry collision cylinder length=0.02 radius=0.02; visual mesh filename=meshes/long_U.stl
- link moving_tip: geometry collision box size=0.003 0.025 0.02; visual box size=0 0 0
- link section_1: geometry collision cylinder length=0.05 radius=0.02; visual mesh filename=meshes/section_1.stl
- link section_2: geometry collision cylinder length=0.05 radius=0.02; visual mesh filename=meshes/section_2.stl
- link section_3: geometry collision cylinder length=0.05 radius=0.02; visual mesh filename=meshes/section_3.stl
- link section_4: geometry collision cylinder length=0.03 radius=0.02; visual mesh filename=meshes/section_4.stl
- link section_5: geometry visual mesh filename=meshes/gripper.stl
